File: Schematics/ece411_schemas/valve_indicator.sch (EAGLE design)
At the start: 66 parts, among them IC1 STM32F042K6T6, T1 2N2222, T2 2N2222, T3 2N2222, T4 2N2222, U1 DIODES_INC._AZ34063UMTR-G1DIO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, U2 DIODES_INC._AZ34063UMTR-G1DIO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

Commit message: dru added, added attributes
Parts:
- RS_L: device SparkFun-Resistors:RESISTOR0603 -> rcl:R-US_R0603
Changed lines of the file:
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@@
 <part name="GND29" library="supply1" library_urn="urn:adsk.eagle:library:371" deviceset="GND" device=""/>
 <part name="GND30" library="supply1" library_urn="urn:adsk.eagle:library:371" deviceset="GND" device=""/>
-<part name="RS_L" library="SparkFun-Resistors" library_urn="urn:adsk.eagle:library:532" deviceset="RESISTOR" device="0603" package3d_urn="urn:adsk.eagle:package:39650/1" value=".33"/>
 <part name="C1" library="rcl" library_urn="urn:adsk.eagle:library:334" deviceset="C-US" device="C0603" package3d_urn="urn:adsk.eagle:package:23616/2" value="4.7nF">
 <spice>
@@
 <part name="R1_L" library="rcl" library_urn="urn:adsk.eagle:library:334" deviceset="R-US_" device="R0603" package3d_urn="urn:adsk.eagle:package:23555/3" value="4.7k"/>
 <part name="R2_L" library="rcl" library_urn="urn:adsk.eagle:library:334" deviceset="R-US_" device="R0603" package3d_urn="urn:adsk.eagle:package:23555/3" value="2.5k"/>
+<part name="RS_L" library="rcl" library_urn="urn:adsk.eagle:library:334" deviceset="R-US_" device="R0603" package3d_urn="urn:adsk.eagle:package:23555/3" value=".33"/>
 </parts>
 <sheets>
@@
 <attribute name="VALUE" x="309.88" y="106.68" size="1.778" layer="96" rot="R180"/>
 </instance>
-<instance part="RS_L" gate="G$1" x="132.08" y="223.52" smashed="yes">
-<attribute name="NAME" x="132.08" y="225.044" size="1.778" layer="95" font="vector" align="bottom-center"/>
-<attribute name="VALUE" x="132.08" y="221.996" size="1.778" layer="96" font="vector" align="top-center"/>
-</instance>
 <instance part="POE_IN" gate="G$1" x="78.74" y="210.82" smashed="yes">
 <attribute name="NAME" x="73.66" y="215.9" size="1.27" layer="95"/>
@@
 <attribute name="NAME" x="240.03" y="230.0986" size="1.778" layer="95"/>
 <attribute name="VALUE" x="240.03" y="225.298" size="1.778" layer="96"/>
+</instance>
+<instance part="RS_L" gate="G$1" x="132.08" y="223.52" smashed="yes">
+<attribute name="NAME" x="128.27" y="225.0186" size="1.778" layer="95"/>
+<attribute name="VALUE" x="128.27" y="220.218" size="1.778" layer="96"/>
 </instance>
 </instances>
@@
 <wire x1="121.92" y1="223.52" x2="127" y2="223.52" width="0.1524" layer="91"/>
 <wire x1="109.22" y1="198.12" x2="109.22" y2="213.36" width="0.1524" layer="91"/>
-<pinref part="RS_L" gate="G$1" pin="1"/>
 <wire x1="81.28" y1="213.36" x2="109.22" y2="213.36" width="0.1524" layer="91"/>
 <junction x="109.22" y="213.36"/>
@@
 <pinref part="C1_H" gate="G$1" pin="1"/>
 <pinref part="RS_H" gate="G$1" pin="1"/>
-</segment>
-</net>
+<pinref part="RS_L" gate="G$1" pin="1"/>
+</segment>
+</net>

Commit message: created bom, finished attributes
Parts:
- C1_H, C1_L: device rcl:C-USC0603 -> rcl:C-US025-025X050; DIS (none) -> Digi-Key; DPN (none) -> 2616-RXW101M1HBK-0811S1-ND; MFR (none) -> SURGE; MPN (none) -> RXW101M1HBK-0811S
- C2_H, C2_L: DIS (none) -> Digi-Key; DPN (none) -> 1292-1438-1-ND; MFR (none) -> Walsin Technology Corporation; MPN (none) -> 0603B471K500CT
- C3_H, C3_L: DIS (none) -> Digi-Key; DPN (none) -> 399-15683-ND; MFR (none) -> KEMET; MPN (none) -> ESH477M050AH4AA
- D1: DIS (none) -> Digi-Key; DPN (none) -> 1N5819GOS-ND; MFR (none) -> On Semiconductor
- D2: DIS (none) -> Digi-Key; DPN (none) -> 1N5819GOS-ND; MFR (none) -> ON Semiconductor
- IC1: MFG STMicroelectronics -> (none); MFR (none) -> STMicroelectronics
- L1, L2: device eagle-ltspice:L0207/10 -> rcl:L-US0204/5; DIS (none) -> Digi-Key; DPN (none) -> AIUR-06-221K-ND; MFR (none) -> Abracon LLC; MPN (none) -> AIUR-06-221K
- R1_H: DIS (none) -> Digi-Key; DPN (none) -> 311-3.30KHRCT-ND; MFR (none) -> Yageo; MPN (none) -> RC0603FR-073K3L
- R1_L: DIS (none) -> Digi-Key; DPN (none) -> RMCF0603FT4K70CT-ND; MFR (none) -> Stackpole Electronics Inc; MPN (none) -> RMCF0603FT4K70
- R2_H: DIS (none) -> Digi-Key; DPN (none) -> A129684CT-ND; MFR (none) -> TE Connectivity Passive Product; MPN (none) -> CRGCQ0603F470R
- R2_L: DIS (none) -> Digi-Key; DPN (none) -> RNCP0603FTD2K49CT-ND; MFR (none) -> Stackpole Electronics Inc; MPN (none) -> RNCP0603FTD2K49
- RS_H, RS_L: DIS (none) -> Digi-Key; DPN (none) -> P.33AJCT-ND; MFR (none) -> Panasonic Electronic Components; MPN (none) -> ERJ-3RQFR33V
Other:
- moved on the sheet: H1, H2, H3, H5

Commit message: updated board bom
Parts:
- C1_H, C1_L: DPN 2616-RXW101M1HBK-0811S1-ND -> 1572-1044-ND; MFR SURGE -> Illinois Capacitor; MPN RXW101M1HBK-0811S -> 107CKR050M
Changed lines of the file:
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@@
 </spice>
 <attribute name="DIS" value="Digi-Key"/>
-<attribute name="DPN" value="2616-RXW101M1HBK-0811S1-ND"/>
-<attribute name="MFR" value="SURGE"/>
-<attribute name="MPN" value="RXW101M1HBK-0811S"/>
+<attribute name="DPN" value="1572-1044-ND"/>
+<attribute name="MFR" value="Illinois Capacitor"/>
+<attribute name="MPN" value="107CKR050M"/>
 </part>
 <part name="C1_H" library="rcl" library_urn="urn:adsk.eagle:library:334" deviceset="C-US" device="025-025X050" package3d_urn="urn:adsk.eagle:package:23629/2" value="100uF">
@@
 </spice>
 <attribute name="DIS" value="Digi-Key"/>
-<attribute name="DPN" value="2616-RXW101M1HBK-0811S1-ND"/>
-<attribute name="MFR" value="SURGE"/>
-<attribute name="MPN" value="RXW101M1HBK-0811S"/>
+<attribute name="DPN" value="1572-1044-ND"/>
+<attribute name="MFR" value="Illinois Capacitor"/>
+<attribute name="MPN" value="107CKR050M"/>
 </part>
 </parts>
