File: Schematics/ece411_schemas/valve_indicator.brd (EAGLE design)
At the start: 85.1 x 53.6 mm, 87 parts, among them Q1 PMV45EN2R, Q2 PMV45EN2R, Q3 PMV45EN2R, Q4 PMV45EN2R, U1 AZ34063UMTR-G1, U2 AZ34063UMTR-G1, U3 STM32F042K6

Commit message: corrections to board
Parts:
- C3_H, C3_L: device rcl:C0603 -> rcl:C025-025X050
- moved D3 1.91 mm to (26.5, 48.4)
- moved C3_L 0.51 mm to (24.8, 44.3)
- moved TP10V 0.40 mm to (44.3, 38.5)
- moved C3_H 0.25 mm to (45.6, 34.7)
Routing:
- net POE: track 79.3 -> 81.2 mm
- net N$16: track 28.8 -> 30.5 mm
- net +10V: track 229.7 -> 230.4 mm
- net GND: track 43.3 -> 42.6 mm
Other:
- board text added: "Jennifer Jordan, Seth Rohrbach, Katie Loseke, Tiffani Shilts Hartman"
- board text removed: "Jennifer Jordan, Seth Rorhbach, Tiffani Hartman-Shilts, Katie Loseke"

Commit message: updates to spacing on boards
Parts:
- turned D1 to 0 degrees
- turned D2 to 0 degrees
Connections:
- removed net N$21: D2.2, L2.1, U2.2
- new net N$10: D2.1, L2.1, U2.2
- net GND: now also D1.2, D2.2; no longer D1.1, D2.1
- net N$5: now also D1.1; no longer D1.2
Routing:
- net N$21: track 47.1 -> 0.00 mm, vias 1 -> 0
- net N$10: track 0.00 -> 45.5 mm, vias 0 -> 1
- net N$5: track 25.0 -> 23.6 mm, vias 0 -> 1
Changed lines of the file:
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@@
 </autorouter>
 <elements>
-<element name="D1" library="On Semiconductor - 1N5819G" package="ON_SEMICONDUCTOR_1N5819G_0" value="1N5819G_0_0" x="58.674" y="37.465" smashed="yes" rot="R180">
-<attribute name="DIS" value="Digi-Key" x="58.674" y="37.465" size="1.778" layer="27" rot="R180" display="off"/>
-<attribute name="DPN" value="1N5819GOS-ND" x="58.674" y="37.465" size="1.778" layer="27" rot="R180" display="off"/>
-<attribute name="MFR" value="On Semiconductor" x="58.674" y="37.465" size="1.778" layer="27" rot="R180" display="off"/>
-<attribute name="MPN" value="1N5819G" x="39.624" y="85.725" size="1.778" layer="27" rot="R180" display="off"/>
-<attribute name="NAME" x="59.25" y="37.941" size="1" layer="25" rot="R180"/>
-</element>
-<element name="D2" library="On Semiconductor - 1N5819G" package="ON_SEMICONDUCTOR_1N5819G_0" value="1N5819G_0_0" x="76.2" y="35.179" smashed="yes" rot="R180">
-<attribute name="DIS" value="Digi-Key" x="76.2" y="35.179" size="1.778" layer="27" rot="R180" display="off"/>
-<attribute name="DPN" value="1N5819GOS-ND" x="76.2" y="35.179" size="1.778" layer="27" rot="R180" display="off"/>
-<attribute name="MFR" value="On Semiconductor" x="76.2" y="35.179" size="1.778" layer="27" rot="R180" display="off"/>
-<attribute name="MPN" value="1N5819G" x="43.18" y="83.439" size="1.778" layer="27" rot="R180" display="off"/>
-<attribute name="NAME" x="76.395" y="35.655" size="1" layer="25" rot="R180"/>
+<element name="D1" library="On Semiconductor - 1N5819G" package="ON_SEMICONDUCTOR_1N5819G_0" value="1N5819G_0_0" x="58.674" y="37.465" smashed="yes">
+<attribute name="DIS" value="Digi-Key" x="58.674" y="37.465" size="1.778" layer="27" display="off"/>
+<attribute name="DPN" value="1N5819GOS-ND" x="58.674" y="37.465" size="1.778" layer="27" display="off"/>
+<attribute name="MFR" value="On Semiconductor" x="58.674" y="37.465" size="1.778" layer="27" display="off"/>
+<attribute name="MPN" value="1N5819G" x="77.724" y="-10.795" size="1.778" layer="27" display="off"/>
+<attribute name="NAME" x="58.098" y="36.989" size="1" layer="25"/>
+</element>
+<element name="D2" library="On Semiconductor - 1N5819G" package="ON_SEMICONDUCTOR_1N5819G_0" value="1N5819G_0_0" x="76.2" y="35.179" smashed="yes">
+<attribute name="DIS" value="Digi-Key" x="76.2" y="35.179" size="1.778" layer="27" display="off"/>
+<attribute name="DPN" value="1N5819GOS-ND" x="76.2" y="35.179" size="1.778" layer="27" display="off"/>
+<attribute name="MFR" value="On Semiconductor" x="76.2" y="35.179" size="1.778" layer="27" display="off"/>
+<attribute name="MPN" value="1N5819G" x="109.22" y="-13.081" size="1.778" layer="27" display="off"/>
+<attribute name="NAME" x="76.005" y="34.703" size="1" layer="25"/>
 </element>
 <element name="HES1" library="pinhead" library_urn="urn:adsk.eagle:library:325" package="1X03" package3d_urn="urn:adsk.eagle:package:22458/2" value="HES1" x="10.16" y="5.08" smashed="yes">
@@
 <contactref element="HES2" pad="2"/>
 <contactref element="U1" pad="4"/>
-<contactref element="D1" pad="1"/>
 <contactref element="U2" pad="4"/>
-<contactref element="D2" pad="1"/>
 <contactref element="C2" pad="2"/>
 <contactref element="C3" pad="2"/>
@@
 <via x="61.468" y="26.924" extent="1-16" drill="0.35"/>
 <via x="58.42" y="28.575" extent="1-16" drill="0.35"/>
+<contactref element="D1" pad="2"/>
+<contactref element="D2" pad="2"/>
 <wire x1="71.12" y1="44.577" x2="74.295" y2="48.768" width="0" layer="19" extent="1-1"/>
 <wire x1="69.215" y1="40.64" x2="71.12" y2="44.577" width="0" layer="19" extent="1-1"/>
@@
 <wire x1="24.765" y1="37.045" x2="24.765" y2="39.155" width="0.3048" layer="1"/>
 </signal>
-<signal name="N$5">
-<contactref element="D1" pad="2"/>
-<contactref element="L1" pad="1"/>
-<contactref element="U1" pad="2"/>
-<wire x1="39.349" y1="32.364" x2="38.058" y2="33.655" width="0.3048" layer="1"/>
-<wire x1="38.058" y1="33.655" x2="37.423" y2="33.655" width="0.3048" layer="1"/>
-<wire x1="53.904" y1="37.465" x2="52.705" y2="37.465" width="0.3048" layer="1"/>
-<wire x1="52.705" y1="37.465" x2="47.604" y2="32.364" width="0.3048" layer="1"/>
-<wire x1="47.604" y1="32.364" x2="39.349" y2="32.364" width="0.3048" layer="1"/>
-<wire x1="53.904" y1="37.465" x2="53.904" y2="38.735" width="0.3048" layer="1"/>
-<wire x1="50.292" y1="41.148" x2="51.491" y2="41.148" width="0.3048" layer="1"/>
-<wire x1="53.904" y1="38.735" x2="51.491" y2="41.148" width="0.3048" layer="1"/>
-</signal>
 <signal name="N$18">
 <contactref element="U2" pad="7"/>
@@
 <wire x1="45.72" y1="46.355" x2="45.3" y2="46.355" width="0.3048" layer="1"/>
 <wire x1="46.355" y1="40.005" x2="46.355" y2="45.72" width="0.3048" layer="1"/>
-</signal>
-<signal name="N$21">
-<contactref element="D2" pad="2"/>
-<contactref element="L2" pad="1"/>
-<contactref element="U2" pad="2"/>
-<wire x1="71.43" y1="35.179" x2="67.874" y2="35.179" width="0.3048" layer="1"/>
-<wire x1="67.874" y1="35.179" x2="59.69" y2="43.363" width="0.3048" layer="1"/>
-<wire x1="59.69" y1="46.101" x2="59.69" y2="43.363" width="0.3048" layer="1"/>
-<wire x1="32.427" y1="41.275" x2="34.29" y2="41.275" width="0.3048" layer="1"/>
-<via x="34.29" y="41.275" extent="1-16" drill="0.35"/>
-<wire x1="34.29" y1="41.275" x2="43.1568375" y2="41.275" width="0.3048" layer="16"/>
-<wire x1="43.1568375" y1="41.275" x2="44.7824375" y2="42.9006" width="0.3048" layer="16"/>
-<wire x1="44.7824375" y1="42.9006" x2="44.8287625" y2="42.9006" width="0.3048" layer="16"/>
-<wire x1="48.0291625" y1="46.101" x2="59.69" y2="46.101" width="0.3048" layer="16"/>
-<wire x1="44.8287625" y1="42.9006" x2="48.0291625" y2="46.101" width="0.3048" layer="16"/>
 </signal>
 <signal name="POE">
@@
 <wire x1="58.96" y1="36.925" x2="57.531" y2="38.354" width="0.3048" layer="1"/>
 </signal>
+<signal name="N$5">
+<contactref element="U1" pad="2"/>
+<contactref element="D1" pad="1"/>
+<contactref element="L1" pad="1"/>
+<wire x1="53.904" y1="37.465" x2="50.292" y2="41.077" width="0.3048" layer="1"/>
+<wire x1="50.292" y1="41.077" x2="50.292" y2="41.148" width="0.3048" layer="1"/>
+<wire x1="50.292" y1="41.148" x2="48.768" y2="41.148" width="0.3048" layer="16"/>
+<wire x1="48.768" y1="41.148" x2="43.18" y2="35.56" width="0.3048" layer="16"/>
+<wire x1="43.18" y1="35.56" x2="43.18" y2="33.147" width="0.3048" layer="16"/>
+<wire x1="43.18" y1="33.147" x2="42.418" y2="32.385" width="0.3048" layer="16"/>
+<wire x1="42.418" y1="32.385" x2="40.894" y2="32.385" width="0.3048" layer="16"/>
+<via x="40.894" y="32.385" extent="1-16" drill="0.35"/>
+<wire x1="40.894" y1="32.385" x2="39.497" y2="32.385" width="0.3048" layer="1"/>
+<wire x1="38.227" y1="33.655" x2="37.423" y2="33.655" width="0.3048" layer="1"/>
+<wire x1="39.497" y1="32.385" x2="38.227" y2="33.655" width="0.3048" layer="1"/>
+</signal>
+<signal name="N$10">
+<contactref element="U2" pad="2"/>
+<contactref element="D2" pad="1"/>
+<contactref element="L2" pad="1"/>
+<wire x1="71.43" y1="35.179" x2="60.508" y2="46.101" width="0.3048" layer="1"/>
+<wire x1="60.508" y1="46.101" x2="59.69" y2="46.101" width="0.3048" layer="1"/>
+<wire x1="32.427" y1="41.275" x2="34.417" y2="41.275" width="0.3048" layer="1"/>
+<via x="34.417" y="41.275" extent="1-16" drill="0.35"/>
+<wire x1="34.417" y1="41.275" x2="35.687" y2="42.545" width="0.3048" layer="16"/>
+<wire x1="54.61" y1="42.545" x2="58.166" y2="46.101" width="0.3048" layer="16"/>
+<wire x1="58.166" y1="46.101" x2="59.69" y2="46.101" width="0.3048" layer="16"/>
+<wire x1="35.687" y1="42.545" x2="54.61" y2="42.545" width="0.3048" layer="16"/>
+</signal>
 </signals>
